Commit message: refs#5 add collision attribute to models

File: src/process_visualiser/urdf/brick_wp_large.urdf (robot description, URDF)
Before this commit: robot brick_wp_large, 2 links, 1 joints
Links:
- link brick_wp_large_origin: geometry collision mesh filename=package://process_visualiser/resources/meshes_resized/brick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 scale=1 1 1; visual mesh filename=package://process_visualiser/resources/meshes_resized/brick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 scale=1 1 1

File: src/process_visualiser/urdf/brick_wp_small.urdf (robot description, URDF)
Before this commit: robot brick_wp_small, 2 links, 1 joints
Links:
- link brick_wp_small_origin: geometry collision mesh filename=package://process_visualiser/resources/meshes_resized/brick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 scale=1 1 1; visual mesh filename=package://process_visualiser/resources/meshes_resized/brick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 scale=1 1 1

File: src/process_visualiser/urdf/cylindrical_assembly_shelf.urdf (robot description, URDF)
Before this commit: robot cylindrical_assembly_shelf, 2 links, 1 joints
Links:
- link cylindrical_assembly_shelf_origin: geometry collision mesh filename=package://process_visualiser/resources/meshes_resized/cylin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 scale=1 1 1; visual mesh filename=package://process_visualiser/resources/meshes_resized/cylin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 scale=1 1 1

File: src/process_visualiser/urdf/cylindrical_wp_large.urdf (robot description, URDF)
Before this commit: robot cylindrical_wp_large, 2 links, 1 joints
Links:
- link cylindrical_wp_large_origin: geometry collision mesh filename=package://process_visualiser/resources/meshes_resized/cylin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 scale=1 1 1; visual mesh filename=package://process_visualiser/resources/meshes_resized/cylin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 scale=1 1 1

File: src/process_visualiser/urdf/cylindrical_wp_small.urdf (robot description, URDF)
Before this commit: robot cylindrical_wp_small, 2 links, 1 joints
Links:
- link cylindrical_wp_small_origin: geometry collision mesh filename=package://process_visualiser/resources/meshes_resized/cylin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 scale=1 1 1; visual mesh filename=package://process_visualiser/resources/meshes_resized/cylin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 scale=1 1 1

File: src/process_visualiser/urdf/robot_table.urdf (robot description, URDF)
Before this commit: robot robot_table, 2 links, 1 joints
Links:
- link robot_table_origin: geometry collision mesh filename=package://process_visualiser/resources/meshes_resized/robot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 scale=1 1 1; visual mesh filename=package://process_visualiser/resources/meshes_resized/robot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 scale=1 1 1

File: src/process_visualiser/urdf/wp_placement_table.urdf (robot description, URDF)
Before this commit: robot wp_placement_table, 2 links, 1 joints
Links:
- link wp_placement_table_origin: geometry collision mesh filename=package://process_visualiser/resources/meshes_resized/wp_pl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 scale=1 1 1; visual mesh filename=package://process_visualiser/resources/meshes_resized/wp_pl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 scale=1 1 1
